File: KiCAD_Project/Orientation_Paddle.kicad_sch (KiCad schematic)
At the start: 45 parts, among them J1 1-0001205, J2 1-0001156, J3 1-0001156, J4 NP_Conn_01x02_Relief, J5 NP_Conn_01x02_Relief, J6 NP_Conn_01x04, J7 NP_Conn_01x02, Q1 1-0001670, U1 1-0001471, U2 1-0000207, Y1 1-0000721

Commit message: Rev 2.2 Changes: - Issue #2 (Swapped to Push Push SD Holder) - Updated PCB and Revision Numbers - Fixed all DRC/ERC Issues
Parts:
- PCB1: Internal Part Number 3-0000273 -> 3-0000299
Changed lines of the file:
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@@
 	(title_block
 		(title "Orientation Paddle")
-		(date "2025-07-03")
-		(rev "2.1.0")
+		(date "2026-02-13")
+		(rev "2.2.0")
 		(company "Leeman Geophysical LLC")
 		(comment 1 "(479) 373-3736")
@@
 			)
 		)
-		(property "Internal Part Number" "3-0000273"
+		(property "Internal Part Number" "3-0000299"
 			(at 164.465 168.91 0)
 			(effects
